File: e75-2g4m10s.brd (EAGLE design)
At the start: 25.4 x 45.1 mm, 30 parts, among them J5 TYPE-C-31-M-12, Q3 SI2323DS, U1 E73-2G4M04S1BE75-2G4M10S, U2 3.3V, U3 CH340E_MSOP10

Commit message: Add files via upload
Parts:
- removed BTN1: (no value), SparkFun-Switches:TACTILE_SWITCH_SMD_4.6X2.8MM
- added BTN: (no value), SparkFun-Switches:TACTILE_SWITCH_SMD_4.6X2.8MM
- moved RST 6.50 mm to (20.7, 3.00)
Connections:
- net DIO17: now also BTN.3, BTN.4; no longer BTN1.3, BTN1.4
- net GND: now also BTN.1, BTN.2; no longer BTN1.1, BTN1.2
Routing:
- net RST: track 29.8 -> 41.4 mm, vias 1 -> 0
- net DIO17: track 47.8 -> 38.2 mm
- net DIO10: track 18.8 -> 17.0 mm
- net DIO9: track 20.6 -> 19.7 mm
- net DIO8: track 23.7 -> 22.8 mm
- net GND: vias 23 -> 24
