File: e75-2g4m10s.sch (EAGLE design)
At the start: 30 parts, among them J5 TYPE-C-31-M-12, Q3 SI2323DS, U1 E73-2G4M04S1BE75-2G4M10S, U2 3.3V, U3 CH340E_MSOP10

Commit message: Add files via upload
Parts:
- renumbered BTN1 to BTN
Changed lines of the file:
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@@
 <part name="GND3" library="supply1" library_urn="urn:adsk.eagle:library:371" deviceset="GND" device=""/>
 <part name="BOOT" library="SparkFun-Switches" library_urn="urn:adsk.eagle:library:535" deviceset="MOMENTARY-SWITCH-SPST-2" device="-SMD-4.6X2.8MM" package3d_urn="urn:adsk.eagle:package:40176/1"/>
-<part name="BTN1" library="SparkFun-Switches" library_urn="urn:adsk.eagle:library:535" deviceset="MOMENTARY-SWITCH-SPST-2" device="-SMD-4.6X2.8MM" package3d_urn="urn:adsk.eagle:package:40176/1"/>
+<part name="BTN" library="SparkFun-Switches" library_urn="urn:adsk.eagle:library:535" deviceset="MOMENTARY-SWITCH-SPST-2" device="-SMD-4.6X2.8MM" package3d_urn="urn:adsk.eagle:package:40176/1"/>
 <part name="D1" library="SparkFun-LED" library_urn="urn:adsk.eagle:library:529" deviceset="LED-RED" device="0603" package3d_urn="urn:adsk.eagle:package:39354/1" value="RED"/>
 <part name="D2" library="SparkFun-LED" library_urn="urn:adsk.eagle:library:529" deviceset="LED-GREEN" device="0603" package3d_urn="urn:adsk.eagle:package:39354/1" value="BLUE"/>
@@
 <attribute name="VALUE" x="307.34" y="25.146" size="1.778" layer="96" font="vector" align="top-center"/>
 </instance>
-<instance part="BTN1" gate="G$1" x="342.9" y="27.94" smashed="yes">
+<instance part="BTN" gate="G$1" x="342.9" y="27.94" smashed="yes">
 <attribute name="NAME" x="342.9" y="32.766" size="1.778" layer="95" font="vector" align="bottom-center"/>
 <attribute name="VALUE" x="342.9" y="25.146" size="1.778" layer="96" font="vector" align="top-center"/>
@@
 </segment>
 <segment>
-<pinref part="BTN1" gate="G$1" pin="1"/>
+<pinref part="BTN" gate="G$1" pin="1"/>
 <wire x1="337.82" y1="27.94" x2="332.74" y2="27.94" width="0.1524" layer="91"/>
 <wire x1="332.74" y1="27.94" x2="332.74" y2="25.4" width="0.1524" layer="91"/>
-<pinref part="BTN1" gate="G$1" pin="2"/>
+<pinref part="BTN" gate="G$1" pin="2"/>
 <wire x1="332.74" y1="25.4" x2="337.82" y2="25.4" width="0.1524" layer="91"/>
 <wire x1="332.74" y1="25.4" x2="332.74" y2="22.86" width="0.1524" layer="91"/>
@@
 </segment>
 <segment>
-<pinref part="BTN1" gate="G$1" pin="3"/>
+<pinref part="BTN" gate="G$1" pin="3"/>
 <wire x1="347.98" y1="27.94" x2="353.06" y2="27.94" width="0.1524" layer="91"/>
 <wire x1="353.06" y1="27.94" x2="353.06" y2="25.4" width="0.1524" layer="91"/>
-<pinref part="BTN1" gate="G$1" pin="4"/>
+<pinref part="BTN" gate="G$1" pin="4"/>
 <wire x1="353.06" y1="25.4" x2="347.98" y2="25.4" width="0.1524" layer="91"/>
 <wire x1="353.06" y1="27.94" x2="360.68" y2="27.94" width="0.1524" layer="91"/>
