File: JN5169_V1/jn5169_v1.sch (EAGLE design)
At the start: 25 parts, among them Y1 32MHZ

Commit message: Add files via upload
Parts:
- added GND, RX, TDO, TX, VCC: TPSTP11R, testpad:TPSTP11R
Connections:
- net DIO6: now also TX.PP
- net DIO7: now also RX.PP
- net GND: now also GND.PP
- net SPIMISO: now also TDO.PP
- net VCC: now also VCC.PP
Changed lines of the file:
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@@
 <part name="Y1" library="ok-xtal-osc-dev" deviceset="48.000MHZ_CX2016DB48000C0FPLC1" device="" value="32MHZ"/>
 <part name="GND3" library="supply1" library_urn="urn:adsk.eagle:library:371" deviceset="GND" device=""/>
+<part name="RX" library="testpad" library_urn="urn:adsk.eagle:library:385" deviceset="TPS" device="TP11R" package3d_urn="urn:adsk.eagle:package:27961/1" value="TPSTP11R"/>
+<part name="TX" library="testpad" library_urn="urn:adsk.eagle:library:385" deviceset="TPS" device="TP11R" package3d_urn="urn:adsk.eagle:package:27961/1" value="TPSTP11R"/>
+<part name="TDO" library="testpad" library_urn="urn:adsk.eagle:library:385" deviceset="TPS" device="TP11R" package3d_urn="urn:adsk.eagle:package:27961/1" value="TPSTP11R"/>
+<part name="VCC" library="testpad" library_urn="urn:adsk.eagle:library:385" deviceset="TPS" device="TP11R" package3d_urn="urn:adsk.eagle:package:27961/1" value="TPSTP11R"/>
+<part name="GND" library="testpad" library_urn="urn:adsk.eagle:library:385" deviceset="TPS" device="TP11R" package3d_urn="urn:adsk.eagle:package:27961/1" value="TPSTP11R"/>
 </parts>
 <sheets>
@@
 <instance part="GND3" gate="1" x="132.08" y="27.94" smashed="yes">
 <attribute name="VALUE" x="129.54" y="25.4" size="1.778" layer="96"/>
+</instance>
+<instance part="RX" gate="G$1" x="220.98" y="78.74" smashed="yes">
+<attribute name="TP_SIGNAL_NAME" x="222.25" y="77.47" size="1.778" layer="97"/>
+</instance>
+<instance part="TX" gate="G$1" x="223.52" y="78.74" smashed="yes">
+<attribute name="TP_SIGNAL_NAME" x="224.79" y="77.47" size="1.778" layer="97"/>
+</instance>
+<instance part="TDO" gate="G$1" x="226.06" y="78.74" smashed="yes">
+<attribute name="TP_SIGNAL_NAME" x="227.33" y="77.47" size="1.778" layer="97"/>
+</instance>
+<instance part="VCC" gate="G$1" x="228.6" y="78.74" smashed="yes">
+<attribute name="TP_SIGNAL_NAME" x="229.87" y="77.47" size="1.778" layer="97"/>
+</instance>
+<instance part="GND" gate="G$1" x="231.14" y="78.74" smashed="yes">
+<attribute name="TP_SIGNAL_NAME" x="232.41" y="77.47" size="1.778" layer="97"/>
 </instance>
 </instances>
@@
 <wire x1="132.08" y1="33.02" x2="132.08" y2="30.48" width="0.1524" layer="91"/>
 <pinref part="GND3" gate="1" pin="GND"/>
+</segment>
+<segment>
+<pinref part="GND" gate="G$1" pin="PP"/>
+<wire x1="231.14" y1="76.2" x2="231.14" y2="66.04" width="0.1524" layer="91"/>
+<label x="231.14" y="66.04" size="1.778" layer="95" rot="R90"/>
 </segment>
 </net>
@@
 <label x="175.26" y="45.72" size="1.778" layer="95" rot="R90"/>
 </segment>
+<segment>
+<pinref part="VCC" gate="G$1" pin="PP"/>
+<wire x1="228.6" y1="76.2" x2="228.6" y2="66.04" width="0.1524" layer="91"/>
+<label x="228.6" y="66.04" size="1.778" layer="95" rot="R90"/>
+</segment>
 </net>
 <net name="N$2" class="0">
@@
 <label x="198.12" y="63.5" size="1.778" layer="95"/>
 </segment>
+<segment>
+<pinref part="TX" gate="G$1" pin="PP"/>
+<wire x1="223.52" y1="76.2" x2="223.52" y2="66.04" width="0.1524" layer="91"/>
+<label x="223.52" y="66.04" size="1.778" layer="95" rot="R90"/>
+</segment>
 </net>
 <net name="DIO7" class="0">
@@
 <wire x1="193.04" y1="66.04" x2="203.2" y2="66.04" width="0.1524" layer="91"/>
 <label x="198.12" y="66.04" size="1.778" layer="95"/>
+</segment>
+<segment>
+<pinref part="RX" gate="G$1" pin="PP"/>
+<wire x1="220.98" y1="76.2" x2="220.98" y2="66.04" width="0.1524" layer="91"/>
+<label x="220.98" y="66.04" size="1.778" layer="95" rot="R90"/>
 </segment>
 </net>
@@
 <label x="154.94" y="109.22" size="1.778" layer="95"/>
 </segment>
-</net>
+<segment>
+<pinref part="TDO" gate="G$1" pin="PP"/>
+<wire x1="226.06" y1="76.2" x2="226.06" y2="66.04" width="0.1524" layer="91"/>
+<label x="226.06" y="66.04" size="1.778" layer="95" rot="R90"/>
+</segment>
+</net>
