File: JN5169_V1/jn5169_v1.brd (EAGLE design)
At the start: 29 x 16.1 mm, 25 parts, among them Y1 32MHZ

Commit message: Add files via upload
Routing:
- net GND: vias 182 -> 184
Changed lines of the file:
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@@
 <text x="15.443" y="3.842" size="0.8128" layer="26" font="vector" ratio="18" rot="MR180">GND</text>
 <text x="23.317" y="6.509" size="0.8128" layer="25" font="vector" ratio="18" rot="SR270">t.me/deaxx</text>
+<wire x1="14.097" y1="8.382" x2="14.605" y2="8.89" width="0.1524" layer="26"/>
+<wire x1="14.605" y1="8.89" x2="14.605" y2="7.874" width="0.1524" layer="26"/>
+<wire x1="14.605" y1="7.874" x2="14.478" y2="8.001" width="0.1524" layer="26"/>
+<wire x1="14.478" y1="8.001" x2="14.097" y2="8.382" width="0.1524" layer="26"/>
+<wire x1="14.097" y1="8.382" x2="14.224" y2="8.382" width="0.1524" layer="26"/>
+<wire x1="14.224" y1="8.382" x2="14.478" y2="8.636" width="0.1524" layer="26"/>
+<wire x1="14.478" y1="8.636" x2="14.478" y2="8.128" width="0.1524" layer="26"/>
+<wire x1="14.478" y1="8.001" x2="14.478" y2="8.128" width="0.1524" layer="26"/>
+<wire x1="14.478" y1="8.128" x2="14.351" y2="8.255" width="0.1524" layer="26"/>
+<wire x1="14.351" y1="8.255" x2="14.351" y2="8.382" width="0.1524" layer="26"/>
 </plain>
 <attributes>
@@
 <via x="2.446" y="14.454" extent="1-16" drill="0.2" diameter="0.45"/>
 <via x="12.939" y="10.434" extent="1-16" drill="0.2" diameter="0.45"/>
+<via x="10.907" y="5.716" extent="1-16" drill="0.2" diameter="0.45"/>
+<via x="12.05" y="8.93" extent="1-16" drill="0.2" diameter="0.45"/>
 </signal>
 <signal name="VCC">

Commit message: Add files via upload
Routing:
- net GND: vias 184 -> 185
Changed lines of the file:
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@@
 <setting verticaltext="up"/>
 </settings>
-<grid distance="0.127" unitdist="mm" unit="mm" style="lines" multiple="1" display="yes" altdistance="5" altunitdist="mil" altunit="mm"/>
+<grid distance="0.003125" unitdist="mic" unit="mm" style="lines" multiple="1" display="yes" altdistance="5" altunitdist="mil" altunit="mm"/>
 <layers>
 <layer number="1" name="Top" color="4" fill="1" visible="yes" active="yes"/>
@@
 </element>
 <element name="C18" library="ok-discretes-dev" package="_PKG_C_0402" value="1p2F" x="15.358" y="13.2772" smashed="yes" rot="R180">
-<attribute name="NAME" x="16.3105" y="13.0232" size="0.762" layer="25" font="vector" ratio="10"/>
+<attribute name="NAME" x="14.5325" y="13.7852" size="0.762" layer="25" font="vector" ratio="10"/>
 <attribute name="VALUE" x="16.247" y="14.2932" size="0.762" layer="27" font="vector" ratio="10" rot="R180"/>
 </element>
@@
 <attribute name="MF" value="Yageo" x="13.9827" y="10.7696" size="1.778" layer="27" rot="R270" display="off"/>
 <attribute name="MP" value="RC0402FR-073M6L" x="13.9827" y="10.7696" size="1.778" layer="27" rot="R270" display="off"/>
-<attribute name="NAME" x="13.3173" y="11.9228" size="0.762" layer="25"/>
+<attribute name="NAME" x="13.4443" y="10.2718" size="0.762" layer="25" rot="R90"/>
 <attribute name="PACKAGE" value="1005 Panasonic Electronic Components" x="13.9827" y="10.7696" size="1.778" layer="27" rot="R270" display="off"/>
 <attribute name="PRICE" value="None" x="13.9827" y="10.7696" size="1.778" layer="27" rot="R270" display="off"/>
@@
 <attribute name="MF" value="Yageo" x="14.8564" y="7.2083" size="1.778" layer="27" rot="R90" display="off"/>
 <attribute name="MP" value="RC0402FR-073M6L" x="14.8564" y="7.2083" size="1.778" layer="27" rot="R90" display="off"/>
-<attribute name="NAME" x="14.1849" y="8.1696" size="0.762" layer="25"/>
+<attribute name="NAME" x="14.5659" y="8.2966" size="0.762" layer="25"/>
 <attribute name="PACKAGE" value="1005 Panasonic Electronic Components" x="14.8564" y="7.2083" size="1.778" layer="27" rot="R90" display="off"/>
 <attribute name="PRICE" value="None" x="14.8564" y="7.2083" size="1.778" layer="27" rot="R90" display="off"/>
@@
 <attribute name="MF" value="Yageo" x="15.3924" y="12.2301" size="1.778" layer="27" rot="R180" display="off"/>
 <attribute name="MP" value="RC0402FR-073M6L" x="15.3924" y="12.2301" size="1.778" layer="27" rot="R180" display="off"/>
-<attribute name="NAME" x="16.3932" y="12.0954" size="0.764" layer="25"/>
+<attribute name="NAME" x="13.3452" y="11.8414" size="0.764" layer="25"/>
 <attribute name="PACKAGE" value="1005 Panasonic Electronic Components" x="15.3924" y="12.2301" size="1.778" layer="27" rot="R180" display="off"/>
 <attribute name="PRICE" value="None" x="15.3924" y="12.2301" size="1.778" layer="27" rot="R180" display="off"/>
@@
 <attribute name="MF" value="Yageo" x="13.3543" y="7.5883" size="1.778" layer="27" display="off"/>
 <attribute name="MP" value="RC0402FR-073M6L" x="13.3543" y="7.5883" size="1.778" layer="27" display="off"/>
-<attribute name="NAME" x="14.1569" y="8.9041" size="0.762" layer="25" rot="R180"/>
+<attribute name="NAME" x="14.5379" y="9.0311" size="0.762" layer="25" rot="R180"/>
 <attribute name="PACKAGE" value="1005 Panasonic Electronic Components" x="13.3543" y="7.5883" size="1.778" layer="27" display="off"/>
 <attribute name="PRICE" value="None" x="13.3543" y="7.5883" size="1.778" layer="27" display="off"/>
@@
 </element>
 <element name="R3" library="ok-discretes-dev" package="_PKG_C_0402" value="43K" x="13.334034375" y="5.4390375" smashed="yes">
-<attribute name="NAME" x="14.350034375" y="4.6770375" size="0.762" layer="25" font="vector"/>
+<attribute name="NAME" x="14.350034375" y="4.5500375" size="0.762" layer="25" font="vector"/>
 <attribute name="VALUE" x="12.445034375" y="4.4230375" size="0.508" layer="27" font="vector"/>
 </element>
@@
 <via x="10.907" y="5.716" extent="1-16" drill="0.2" diameter="0.45"/>
 <via x="12.05" y="8.93" extent="1-16" drill="0.2" diameter="0.45"/>
+<via x="15.91610625" y="11.42595625" extent="1-16" drill="0.2" diameter="0.45"/>
 </signal>
 <signal name="VCC">
@@
 <via x="11.684" y="5.08" extent="1-16" drill="0.3"/>
 <wire x1="12.143" y1="4.445" x2="11.303" y2="4.445" width="0.3048" layer="1"/>
-<wire x1="10.414" y1="5.334" x2="9.652" y2="5.334" width="0.3048" layer="1"/>
+<wire x1="9.652" y1="5.334" x2="10.414" y2="5.334" width="0.3048" layer="1"/>
 <wire x1="9.652" y1="5.334" x2="9.275" y2="5.711" width="0.3048" layer="1"/>
 <wire x1="9.275" y1="5.711" x2="9.275" y2="6.171" width="0.3048" layer="1"/>

Commit message: Add files via upload
Parts:
- added GND, RX, TDO, TX, VCC: TPSTP11R, testpad:TP11R
- moved C6 0.48 mm to (3.07, 12.2), turned to 0 degrees
Connections:
- net DIO6: now also TX.TP
- net DIO7: now also RX.TP
- net GND: now also GND.TP
- net SPIMISO: now also TDO.TP
- net VCC: now also VCC.TP
Routing:
- net SPIMISO: track 4.42 -> 16.6 mm, vias 0 -> 1
- net VCC: track 33.1 -> 37.1 mm
- net DIO6: track 8.58 -> 10.6 mm
- net DIO7: track 8.86 -> 10.7 mm
- net GND: track 5.00 -> 5.12 mm, vias 185 -> 184
Other:
- board text added: "ISP"
- board text added: "RX"
- board text added: "TX"
- board text added: "VCC"

Commit message: Add files via upload
Parts:
- moved GND 0.25 mm to (1.77, 12.4)
- moved RX 0.25 mm to (1.74, 8.57)
- moved TDO 0.25 mm to (1.74, 11.1)
- moved TX 0.25 mm to (1.76, 9.84)
- moved VCC 0.25 mm to (1.74, 7.28)
Routing:
- net DIO14: track 13.6 -> 12.4 mm
- net SPIMISO: track 16.6 -> 15.7 mm
- net DIO13: track 11.7 -> 11.0 mm
- net DIO12: track 12.0 -> 11.3 mm
- net GND: track 5.12 -> 5.03 mm, vias 184 -> 188
Other:
- board text added: "."

Commit message: Add files via upload
Parts:
- moved E1 24.3 mm to (1.99, 24.2), turned to 270 degrees
- moved J2 13.9 mm to (2.72, 0.01), turned to 0 degrees
- moved J1 13.1 mm to (0.22, 12.7), turned to 270 degrees
- moved J3 13.1 mm to (16.3, 12.7), turned to 270 degrees
- moved C18 12.4 mm to (3.11, 15.2), turned to 270 degrees
- moved L4 11.6 mm to (4.15, 15.3), turned to 270 degrees
- moved C10 11.2 mm to (14.9, 12.5), turned to 270 degrees
- moved GND 11.0 mm to (4.01, 1.64), turned to 270 degrees
- moved C1 10.2 mm to (5.62, 14.9), turned to 180 degrees
- moved TDO 10.1 mm to (5.27, 1.61), turned to 270 degrees
- moved C7 10.0 mm to (13.9, 12.4), turned to 270 degrees
- moved R1 10.0 mm to (14.9, 10.7), turned to 90 degrees
- moved C16 9.85 mm to (12.9, 2.97), turned to 0 degrees
- moved TX 9.50 mm to (6.54, 1.63), turned to 270 degrees
- moved C3 9.43 mm to (9.17, 14.7), turned to 180 degrees
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Routing:
- net SPIMISO: track 15.7 -> 16.5 mm
Other:
- board size 29 x 16.1 mm -> 16.1 x 29 mm

Commit message: Add files via upload
Parts:
- moved C3 0.05 mm to (9.23, 14.7)
Routing:
- net VCC: track 37.2 -> 47.0 mm, vias 5 -> 7
- net RESET_N: track 15.9 -> 15.3 mm
- net GND: vias 188 -> 189
